File: SMP v.2.kicad_pcb (KiCad board)
At the start: 2 copper layers, 123.8 x 58.7 mm, 17 parts, among them U1 Elite-C

Commit message: update based on 2moon comment
Connections:
- U1 pad 23: Net-(U1-Pad23) -> GND
- U1 pad 3: Net-(U1-Pad3) -> GND
- U1 pad 4: Net-(U1-Pad4) -> GND
Routing:
- net GND: track 0.00 -> 26.9 mm
- added copper zone on B.Cu, net GND
- added copper zone on F.Cu, net GND
