File: SMP v.2.sch (KiCad schematic (older format))
At the start: 17 parts, among them U1 Elite-C

Commit message: update based on 2moon comment
Connections:
- net GND: now reaches U1.23 (GND)
- net GND: now also U1.3 (GND), U1.4 (GND)
Changed lines of the file:
@@
 NoConn ~ 3700 3700
 NoConn ~ 3600 3700
+$Comp
+L power:GND #PWR?
+U 1 1 610C3B30
+P 2900 2400
+F 0 "#PWR?" H 2900 2150 50  0001 C CNN
+F 1 "GND" H 2905 2227 50  0000 C CNN
+F 2 "" H 2900 2400 50  0001 C CNN
+F 3 "" H 2900 2400 50  0001 C CNN
+	1    2900 2400
+	1    0    0    -1
+$EndComp
+$Comp
+L power:GND #PWR?
+U 1 1 610C4A53
+P 4700 2300
+F 0 "#PWR?" H 4700 2050 50  0001 C CNN
+F 1 "GND" H 4705 2127 50  0000 C CNN
+F 2 "" H 4700 2300 50  0001 C CNN
+F 3 "" H 4700 2300 50  0001 C CNN
+	1    4700 2300
+	1    0    0    -1
+$EndComp
+Wire Wire Line
+	2900 2400 3100 2400
+Wire Wire Line
+	3100 2500 3100 2400
+Connection ~ 3100 2400
+Wire Wire Line
+	4700 2300 4500 2300
 $EndSCHEMATC
