File: pcb/SMP v.2.kicad_pcb (KiCad board)
At the start: 2 copper layers, 123.8 x 58.7 mm, 21 parts, among them U1 Elite-C

Commit message: Add BOM and Pos file
Parts:
- MX1, MX2, MX3, MX4, MX5, MX6, MX7, MX8: footprint MX_Alps_Hybrid:MX-1U-NoLED -> MX_Only:MXOnly-1U-NoLED
Connections:
- U1 pad 13: ROW1 -> Net-(U1-Pad13)
- U1 pad 14: ROW0 -> Net-(U1-Pad14)
- U1 pad 7: Net-(U1-Pad7) -> ROW0
- U1 pad 8: Net-(U1-Pad8) -> ROW1
Routing:
- net ROW0: track 94.2 -> 114.6 mm, vias 0 -> 4
- net ROW1: track 108.3 -> 126.3 mm, vias 4 -> 0
- net COL0: track 61.2 -> 57.0 mm
- net COL2: track 109.2 -> 105.0 mm
- net COL3: track 133.2 -> 129.1 mm
- net COL1: track 85.5 -> 81.3 mm
Other:
- board text added: "SMP V.2"

Commit message: tidy up the folder
Routing:
- net COL0: track 57.0 -> 58.9 mm
- net COL3: track 129.1 -> 130.9 mm
- net COL2: track 105.0 -> 106.6 mm
- net COL1: track 81.3 -> 82.8 mm
- net Net-(D8-Pad2): track 30.8 -> 29.6 mm
- net Net-(D7-Pad2): track 31.5 -> 30.3 mm
- net Net-(D5-Pad2): track 30.8 -> 29.6 mm
- net Net-(D6-Pad2): track 31.6 -> 30.5 mm
- net ROW1: track 126.3 -> 126.9 mm

Commit message: WIP: on board mcu
Parts:
- removed ? (x3), REF**: MountingHole_2.2mm_M2_Pad, MountingHole:MountingHole_2.2mm_M2_Pad
- added C1: 1uF, Capacitor_SMD:C_0805_2012Metric, F.Cu at (64.3, 44.5)
- added C2: 0.1uF, Capacitor_SMD:C_0805_2012Metric, F.Cu at (53.8, 53.6)
- added C3: 0.1uF, Capacitor_SMD:C_0805_2012Metric, F.Cu at (53.8, 55.8)
- added C4: 0.1uF, Capacitor_SMD:C_0805_2012Metric, F.Cu at (57.7, 44.5)
- added C5: 10uF, Capacitor_SMD:C_0805_2012Metric, F.Cu at (53.8, 58.2)
- added F1: 500mA, Fuse:Fuse_1206_3216Metric, F.Cu at (54.1, 44.0)
- added H1: MountingHole_Pad, MountingHole:MountingHole_3.2mm_M3_Pad, F.Cu at (150.9, 30.4)
- added H2: MountingHole_Pad, MountingHole:MountingHole_3.2mm_M3_Pad, F.Cu at (150.9, 78.8)
- added H3: MountingHole_Pad, MountingHole:MountingHole_3.2mm_M3_Pad, F.Cu at (46.5, 30.4)
- added H4: MountingHole_Pad, MountingHole:MountingHole_3.2mm_M3_Pad, F.Cu at (46.5, 78.8)
- added J1: USB_C_Receptacle_USB2.0, Connector_USB:USB_C_Receptacle_HRO_TYPE-C-31-M-12, F.Cu at (61.1, 29.5)
- added R1: 10k, Resistor_SMD:R_0805_2012Metric, F.Cu at (55.2, 63.0)
- added R2: 22, Resistor_SMD:R_0805_2012Metric, F.Cu at (61.9, 44.5)
- added R3: 22, Resistor_SMD:R_0805_2012Metric, F.Cu at (60.0, 44.5)
- added R4: 5.1k, Resistor_SMD:R_0805_2012Metric, F.Cu at (63.8, 40.3)
- added R5: 5.1k, Resistor_SMD:R_0805_2012Metric, F.Cu at (58.0, 40.3)
- added R6: 10k, Resistor_SMD:R_0805_2012Metric, F.Cu at (61.2, 59.3)
- added SW1: SW_Push, random-keyboard-parts:SKQG-1155865, F.Cu at (61.6, 64.9)
- added Y1: 16MHz, Crystal:Resonator_SMD_muRata_CSTxExxV-3Pin_3.0x1.1mm, F.Cu at (53.4, 50.4)
- U1: value Elite-C -> ATmega32U2-AU; footprint Keebio-Parts:Elite-C -> Package_QFP:TQFP-32_7x7mm_P0.8mm
- moved D2 38.3 mm to (131.6, 31.7)
- moved D3 28.5 mm to (83.9, 31.7)
- moved D7 18.8 mm to (103.0, 31.7)
- moved D8 18.8 mm to (122.1, 31.7)
- moved U1 10.4 mm to (61.7, 52.8), turned to 0 degrees
- moved D4 9.82 mm to (141.2, 31.7)
- moved D5 9.65 mm to (93.4, 31.7)
- moved D6 9.63 mm to (112.5, 31.7)
- moved D1 0.14 mm to (74.3, 31.7)
Connections:
- D1 pad 1: ROW0 -> ROW1
- D2 pad 1: ROW0 -> ROW1
- D7 pad 1: ROW1 -> ROW0
- D8 pad 1: ROW1 -> ROW0
- MX2 pad 2: Net-(D2-Pad2) -> Net-(D5-Pad2)
- MX3 pad 2: Net-(D3-Pad2) -> Net-(D6-Pad2)
- MX4 pad 2: Net-(D4-Pad2) -> Net-(D2-Pad2)
- MX5 pad 2: Net-(D5-Pad2) -> Net-(D3-Pad2)
- MX6 pad 2: Net-(D6-Pad2) -> Net-(D7-Pad2)
- MX7 pad 2: Net-(D7-Pad2) -> Net-(D8-Pad2)
- MX8 pad 2: Net-(D8-Pad2) -> Net-(D4-Pad2)
- U1 pad 10: COL2 -> Net-(U1-Pad10)
- U1 pad 11: COL1 -> Net-(U1-Pad11)
- U1 pad 12: COL0 -> Net-(U1-Pad12)
- U1 pad 18: Net-(U1-Pad18) -> COL0
- U1 pad 19: Net-(U1-Pad19) -> COL1
- U1 pad 20: Net-(U1-Pad20) -> COL2
- U1 pad 21: Net-(U1-Pad21) -> COL3
- U1 pad 23: GND -> Net-(U1-Pad23)
- U1 pad 25: Net-(U1-Pad25) -> ROW0
- U1 pad 26: Net-(U1-Pad26) -> ROW1
- U1 pad 28: Net-(U1-Pad28) -> GND
- U1 pad 4: GND -> +5V
- U1 pad 7: ROW0 -> Net-(U1-Pad7)
- U1 pad 8: ROW1 -> Net-(U1-Pad8)
- U1 pad 9: COL3 -> Net-(U1-Pad9)
Routing:
- net Net-(R1-Pad2): track 0.00 -> 44.8 mm, vias 0 -> 2
- net COL3: track 130.9 -> 89.3 mm, vias 0 -> 1
- net COL2: track 106.6 -> 69.9 mm, vias 0 -> 1
- net ROW1: track 126.9 -> 93.7 mm, vias 0 -> 5
- net COL1: track 82.8 -> 50.6 mm, vias 0 -> 1
- net COL0: track 58.9 -> 31.4 mm, vias 0 -> 1
- net Net-(F1-Pad2): track 0.00 -> 22.2 mm, vias 0 -> 2
- net Net-(D6-Pad2): track 30.5 -> 10.5 mm
- net Net-(D5-Pad2): track 29.6 -> 10.6 mm
- net Net-(D4-Pad2): track 10.7 -> 29.0 mm
- net Net-(D3-Pad2): track 10.6 -> 29.0 mm
- net +5V: track 0.00 -> 17.8 mm
- net ROW0: track 114.5 -> 99.1 mm, vias 4 -> 0
- net D-: track 0.00 -> 13.9 mm, vias 0 -> 2
- net D+: track 0.00 -> 13.2 mm
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Other:
- board size 123.8 x 58.7 mm -> 114.7 x 58.7 mm

Commit message: WIP: on board mcu
Routing:
- net Net-(D3-Pad2): track 29.0 -> 30.5 mm
- net Net-(D8-Pad2): track 29.0 -> 30.4 mm
- net Net-(D7-Pad2): track 29.0 -> 30.4 mm
- net Net-(D4-Pad2): track 29.0 -> 30.4 mm
- net COL1: track 50.6 -> 51.1 mm
- net COL0: track 31.4 -> 32.0 mm
- net COL3: track 89.3 -> 89.8 mm
Changed lines of the file:
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@@
     (thickness 1.6)
     (drawings 26)
-    (tracks 190)
+    (tracks 202)
     (zones 0)
     (modules 36)
@@
   (segment (start 133.286352 34.566752) (end 138.7259 40.0063) (width 0.254) (layer F.Cu) (net 3))
   (segment (start 133.286352 31.73222) (end 133.286352 34.566752) (width 0.254) (layer F.Cu) (net 3))
-  (segment (start 85.546342 55.085858) (end 81.5759 59.0563) (width 0.254) (layer F.Cu) (net 4))
-  (segment (start 85.546342 31.73222) (end 85.546342 55.085858) (width 0.254) (layer F.Cu) (net 4))
-  (segment (start 142.83436 54.94784) (end 138.7259 59.0563) (width 0.254) (layer F.Cu) (net 5))
-  (segment (start 142.83436 31.73222) (end 142.83436 54.94784) (width 0.254) (layer F.Cu) (net 5))
+  (segment (start 87.43188 53.20032) (end 81.5759 59.0563) (width 0.254) (layer F.Cu) (net 4))
+  (segment (start 87.43188 33.617758) (end 87.43188 53.20032) (width 0.254) (layer F.Cu) (net 4))
+  (segment (start 85.546342 31.73222) (end 87.43188 33.617758) (width 0.254) (layer F.Cu) (net 4))
+  (segment (start 144.49806 53.28414) (end 138.7259 59.0563) (width 0.254) (layer F.Cu) (net 5))
+  (segment (start 144.49806 33.39592) (end 144.49806 53.28414) (width 0.254) (layer F.Cu) (net 5))
+  (segment (start 142.83436 31.73222) (end 144.49806 33.39592) (width 0.254) (layer F.Cu) (net 5))
   (via (at 108.92028 29.76372) (size 0.8) (drill 0.4) (layers F.Cu B.Cu) (net 6))
   (segment (start 110.88878 31.73222) (end 108.92028 29.76372) (width 0.254) (layer F.Cu) (net 6))
@@
   (segment (start 69.806818 29.76372) (end 68.225619 31.344919) (width 0.254) (layer B.Cu) (net 6))
   (segment (start 89.84996 29.76372) (end 69.806818 29.76372) (width 0.254) (layer B.Cu) (net 6))
-  (segment (start 75.2259 42.5463) (end 75.2259 61.5963) (width 0.254) (layer F.Cu) (net 7))
   (via (at 68.9102 54.7624) (size 0.8) (drill 0.4) (layers F.Cu B.Cu) (net 7))
   (segment (start 65.9786 54.7624) (end 65.972 54.7558) (width 0.254) (layer F.Cu) (net 7))
@@
   (segment (start 75.2259 61.0781) (end 75.2259 61.5963) (width 0.254) (layer B.Cu) (net 7))
   (segment (start 68.9102 54.7624) (end 75.2259 61.0781) (width 0.254) (layer B.Cu) (net 7))
-  (segment (start 94.2759 42.5463) (end 94.2759 61.5963) (width 0.254) (layer F.Cu) (net 8))
+  (segment (start 75.86726 60.95494) (end 75.2259 61.5963) (width 0.254) (layer F.Cu) (net 7))
+  (segment (start 75.86726 43.18766) (end 75.86726 60.95494) (width 0.254) (layer F.Cu) (net 7))
+  (segment (start 75.2259 42.5463) (end 75.86726 43.18766) (width 0.254) (layer F.Cu) (net 7))
   (segment (start 66.0036 53.9242) (end 65.972 53.9558) (width 0.254) (layer F.Cu) (net 8))
   (via (at 67.88404 53.95976) (size 0.8) (drill 0.4) (layers F.Cu B.Cu) (net 8))
@@
   (segment (start 86.63936 53.95976) (end 94.2759 61.5963) (width 0.254) (layer B.Cu) (net 8))
   (segment (start 67.88404 53.95976) (end 86.63936 53.95976) (width 0.254) (layer B.Cu) (net 8))
-  (segment (start 113.3259 42.5463) (end 113.3259 61.5963) (width 0.254) (layer F.Cu) (net 9))
+  (segment (start 94.95028 60.92192) (end 94.2759 61.5963) (width 0.254) (layer F.Cu) (net 8))
+  (segment (start 94.95028 43.22068) (end 94.95028 60.92192) (width 0.254) (layer F.Cu) (net 8))
+  (segment (start 94.2759 42.5463) (end 94.95028 43.22068) (width 0.254) (layer F.Cu) (net 8))
   (via (at 68.9102 53.15204) (size 0.8) (drill 0.4) (layers F.Cu B.Cu) (net 9))
   (segment (start 65.97576 53.15204) (end 65.972 53.1558) (width 0.254) (layer F.Cu) (net 9))
@@
   (segment (start 104.88164 53.15204) (end 113.3259 61.5963) (width 0.254) (layer B.Cu) (net 9))
   (segment (start 68.88988 53.15204) (end 104.88164 53.15204) (width 0.254) (layer B.Cu) (net 9))
-  (segment (start 132.3759 42.5463) (end 132.3759 61.5963) (width 0.254) (layer F.Cu) (net 10))
+  (segment (start 113.89868 61.02352) (end 113.3259 61.5963) (width 0.254) (layer F.Cu) (net 9))
+  (segment (start 113.89868 43.11908) (end 113.89868 61.02352) (width 0.254) (layer F.Cu) (net 9))
+  (segment (start 113.3259 42.5463) (end 113.89868 43.11908) (width 0.254) (layer F.Cu) (net 9))
   (segment (start 65.972 52.3558) (end 67.80624 52.3558) (width 0.254) (layer F.Cu) (net 10))
   (via (at 67.87134 52.4209) (size 0.8) (drill 0.4) (layers F.Cu B.Cu) (net 10))
@@
   (segment (start 67.80624 52.3558) (end 67.87134 52.4209) (width 0.254) (layer F.Cu) (net 10))
   (segment (start 123.2005 52.4209) (end 67.87134 52.4209) (width 0.254) (layer B.Cu) (net 10))
+  (segment (start 133.0071 43.1775) (end 133.0071 60.9651) (width 0.254) (layer F.Cu) (net 10))
+  (segment (start 133.0071 60.9651) (end 132.3759 61.5963) (width 0.254) (layer F.Cu) (net 10))
+  (segment (start 132.3759 42.5463) (end 133.0071 43.1775) (width 0.254) (layer F.Cu) (net 10))
   (segment (start 55.0864 49.219) (end 53.4162 49.219) (width 0.254) (layer F.Cu) (net 12))
   (segment (start 55.8232 49.9558) (end 55.0864 49.219) (width 0.254) (layer F.Cu) (net 12))
@@
   (segment (start 114.190348 34.520748) (end 119.6759 40.0063) (width 0.254) (layer F.Cu) (net 37))
   (segment (start 114.190348 31.73222) (end 114.190348 34.520748) (width 0.254) (layer F.Cu) (net 37))
-  (segment (start 104.642346 55.039854) (end 100.6259 59.0563) (width 0.254) (layer F.Cu) (net 38))
-  (segment (start 104.642346 31.73222) (end 104.642346 55.039854) (width 0.254) (layer F.Cu) (net 38))
-  (segment (start 123.73835 54.99385) (end 119.6759 59.0563) (width 0.254) (layer F.Cu) (net 39))
-  (segment (start 123.73835 31.73222) (end 123.73835 54.99385) (width 0.254) (layer F.Cu) (net 39))
+  (segment (start 106.35742 53.32478) (end 100.6259 59.0563) (width 0.254) (layer F.Cu) (net 38))
+  (segment (start 106.35742 33.447294) (end 106.35742 53.32478) (width 0.254) (layer F.Cu) (net 38))
+  (segment (start 104.642346 31.73222) (end 106.35742 33.447294) (width 0.254) (layer F.Cu) (net 38))
+  (segment (start 125.476 53.2562) (end 119.6759 59.0563) (width 0.254) (layer F.Cu) (net 39))
+  (segment (start 125.476 33.46987) (end 125.476 53.2562) (width 0.254) (layer F.Cu) (net 39))
+  (segment (start 123.73835 31.73222) (end 125.476 33.46987) (width 0.254) (layer F.Cu) (net 39))
   (segment (start 65.98572 50.76952) (end 65.972 50.7558) (width 0.254) (layer F.Cu) (net 40))
   (segment (start 55.061 51.619) (end 53.4162 51.619) (width 0.254) (layer F.Cu) (net 46))
