File: pcb/SMP v.2.sch (KiCad schematic (older format))
At the start: 17 parts, among them U1 Elite-C

Commit message: Add BOM and Pos file
Parts:
- MX1, MX2, MX3, MX4, MX5, MX6, MX7, MX8: footprint MX_Alps_Hybrid:MX-1U-NoLED -> MX_Only:MXOnly-1U-NoLED; symbol MX_Alps_Hybrid:MX-NoLED -> SMP-v.2-rescue:MX-NoLED-MX_Alps_Hybrid
- U1: symbol keebio:Elite-C -> SMP-v.2-rescue:Elite-C-keebio
Changed lines of the file:
@@
 $EndDescr
 $Comp
-L keebio:Elite-C U1
+L SMP-v.2-rescue:Elite-C-keebio U1
 U 1 1 610873F7
 P 3800 2750
@@
 $EndComp
 $Comp
-L MX_Alps_Hybrid:MX-NoLED MX1
+L SMP-v.2-rescue:MX-NoLED-MX_Alps_Hybrid MX1
 U 1 1 61087E0A
 P 5950 2700
 F 0 "MX1" H 5983 2923 60  0000 C CNN
 F 1 "MX-NoLED" H 5983 2849 20  0000 C CNN
-F 2 "MX_Alps_Hybrid:MX-1U-NoLED" H 5325 2675 60  0001 C CNN
+F 2 "MX_Only:MXOnly-1U-NoLED" H 5325 2675 60  0001 C CNN
 F 3 "" H 5325 2675 60  0001 C CNN
 	1    5950 2700
@@
 $EndComp
 $Comp
-L MX_Alps_Hybrid:MX-NoLED MX2
+L SMP-v.2-rescue:MX-NoLED-MX_Alps_Hybrid MX2
 U 1 1 6108A2CF
 P 6550 2700
 F 0 "MX2" H 6583 2923 60  0000 C CNN
 F 1 "MX-NoLED" H 6583 2849 20  0000 C CNN
-F 2 "MX_Alps_Hybrid:MX-1U-NoLED" H 5925 2675 60  0001 C CNN
+F 2 "MX_Only:MXOnly-1U-NoLED" H 5925 2675 60  0001 C CNN
 F 3 "" H 5925 2675 60  0001 C CNN
 	1    6550 2700
@@
 $EndComp
 $Comp
-L MX_Alps_Hybrid:MX-NoLED MX3
+L SMP-v.2-rescue:MX-NoLED-MX_Alps_Hybrid MX3
 U 1 1 6108B8DB
 P 7150 2700
 F 0 "MX3" H 7183 2923 60  0000 C CNN
 F 1 "MX-NoLED" H 7183 2849 20  0000 C CNN
-F 2 "MX_Alps_Hybrid:MX-1U-NoLED" H 6525 2675 60  0001 C CNN
+F 2 "MX_Only:MXOnly-1U-NoLED" H 6525 2675 60  0001 C CNN
 F 3 "" H 6525 2675 60  0001 C CNN
 	1    7150 2700
@@
 $EndComp
 $Comp
-L MX_Alps_Hybrid:MX-NoLED MX4
+L SMP-v.2-rescue:MX-NoLED-MX_Alps_Hybrid MX4
 U 1 1 6108BA47
 P 7750 2700
 F 0 "MX4" H 7783 2923 60  0000 C CNN
 F 1 "MX-NoLED" H 7783 2849 20  0000 C CNN
-F 2 "MX_Alps_Hybrid:MX-1U-NoLED" H 7125 2675 60  0001 C CNN
+F 2 "MX_Only:MXOnly-1U-NoLED" H 7125 2675 60  0001 C CNN
 F 3 "" H 7125 2675 60  0001 C CNN
 	1    7750 2700
@@
 $EndComp
 $Comp
-L MX_Alps_Hybrid:MX-NoLED MX5
+L SMP-v.2-rescue:MX-NoLED-MX_Alps_Hybrid MX5
 U 1 1 61091781
 P 5950 3400
 F 0 "MX5" H 5983 3623 60  0000 C CNN
 F 1 "MX-NoLED" H 5983 3549 20  0000 C CNN
-F 2 "MX_Alps_Hybrid:MX-1U-NoLED" H 5325 3375 60  0001 C CNN
+F 2 "MX_Only:MXOnly-1U-NoLED" H 5325 3375 60  0001 C CNN
 F 3 "" H 5325 3375 60  0001 C CNN
 	1    5950 3400
@@
 $EndComp
 $Comp
-L MX_Alps_Hybrid:MX-NoLED MX6
+L SMP-v.2-rescue:MX-NoLED-MX_Alps_Hybrid MX6
 U 1 1 6109178D
 P 6550 3400
 F 0 "MX6" H 6583 3623 60  0000 C CNN
 F 1 "MX-NoLED" H 6583 3549 20  0000 C CNN
-F 2 "MX_Alps_Hybrid:MX-1U-NoLED" H 5925 3375 60  0001 C CNN
+F 2 "MX_Only:MXOnly-1U-NoLED" H 5925 3375 60  0001 C CNN
 F 3 "" H 5925 3375 60  0001 C CNN
 	1    6550 3400
@@
 $EndComp
 $Comp
-L MX_Alps_Hybrid:MX-NoLED MX7
+L SMP-v.2-rescue:MX-NoLED-MX_Alps_Hybrid MX7
 U 1 1 61091799
 P 7150 3400
 F 0 "MX7" H 7183 3623 60  0000 C CNN
 F 1 "MX-NoLED" H 7183 3549 20  0000 C CNN
-F 2 "MX_Alps_Hybrid:MX-1U-NoLED" H 6525 3375 60  0001 C CNN
+F 2 "MX_Only:MXOnly-1U-NoLED" H 6525 3375 60  0001 C CNN
 F 3 "" H 6525 3375 60  0001 C CNN
 	1    7150 3400
@@
 $EndComp
 $Comp
-L MX_Alps_Hybrid:MX-NoLED MX8
+L SMP-v.2-rescue:MX-NoLED-MX_Alps_Hybrid MX8
 U 1 1 610917A5
 P 7750 3400
 F 0 "MX8" H 7783 3623 60  0000 C CNN
 F 1 "MX-NoLED" H 7783 3549 20  0000 C CNN
-F 2 "MX_Alps_Hybrid:MX-1U-NoLED" H 7125 3375 60  0001 C CNN
+F 2 "MX_Only:MXOnly-1U-NoLED" H 7125 3375 60  0001 C CNN
 F 3 "" H 7125 3375 60  0001 C CNN
 	1    7750 3400
@@
 Text GLabel 7900 2100 1    50   Input ~ 0
 COL3
-Text GLabel 4500 3300 2    50   Input ~ 0
+Text GLabel 3100 2900 0    50   Input ~ 0
 ROW1
-Text GLabel 4500 3200 2    50   Input ~ 0
+Text GLabel 3100 2800 0    50   Input ~ 0
 ROW0
 Text GLabel 3100 3300 0    50   Input ~ 0
@@
 NoConn ~ 3600 3700
 $Comp
-L power:GND #PWR?
+L power:GND #PWR0101
 U 1 1 610C3B30
 P 2900 2400
-F 0 "#PWR?" H 2900 2150 50  0001 C CNN
+F 0 "#PWR0101" H 2900 2150 50  0001 C CNN
 F 1 "GND" H 2905 2227 50  0000 C CNN
 F 2 "" H 2900 2400 50  0001 C CNN
@@
 $EndComp
 $Comp
-L power:GND #PWR?
+L power:GND #PWR0102
 U 1 1 610C4A53
 P 4700 2300
-F 0 "#PWR?" H 4700 2050 50  0001 C CNN
+F 0 "#PWR0102" H 4700 2050 50  0001 C CNN
 F 1 "GND" H 4705 2127 50  0000 C CNN
 F 2 "" H 4700 2300 50  0001 C CNN

Commit message: wip
Parts:
- removed D5, D6, D7, D8: D_Small, Diode_SMD:D_SOD-123, symbol Device:D_Small
- removed U1: Elite-C, Keebio-Parts:Elite-C, symbol SMP-v.2-rescue:Elite-C-keebio
- added C?: 1uF, symbol Device:C_Small
- added C? (x3): 0.1uF, symbol Device:C_Small
- added C?: 10uF, symbol Device:C_Small
- added C? (x2): 22pF, symbol Device:C_Small
- added R? (x2): 10k, symbol Device:R_Small
- added R? (x2): 22, symbol Device:R_Small
- added SW?: SW_Push, symbol Switch:SW_Push
- added U?: ATmega32U4-AU, Package_QFP:TQFP-44_10x10mm_P0.8mm, symbol MCU_Microchip_ATmega:ATmega32U4-AU
- added Y?: 16MHz, symbol Device:Crystal_GND24_Small
Connections:
- net labels added: +5V, D+, D-
- wire segments 27 -> 65
- no-connect marks 5 -> 0
Other:
- moved on the sheet: D1, D2, D3, D4, MX5, MX6, MX7, MX8

Commit message: WIP: on board mcu
Parts:
- removed C? (x2): 22pF, symbol Device:C_Small
- removed U?: ATmega32U4-AU, Package_QFP:TQFP-44_10x10mm_P0.8mm, symbol MCU_Microchip_ATmega:ATmega32U4-AU
- removed Y?: 16MHz, symbol Device:Crystal_GND24_Small
- added D5, D6, D7, D8: D_Small, Diode_SMD:D_SOD-123, symbol Device:D_Small
- added F1: 500mA, Fuse:Fuse_1206_3216Metric, symbol Device:Polyfuse_Small
- added H1, H2, H3, H4: MountingHole_Pad, MountingHole:MountingHole_3.2mm_M3_Pad, symbol Mechanical:MountingHole_Pad
- added J1: USB_C_Receptacle_USB2.0, Connector_USB:USB_C_Receptacle_HRO_TYPE-C-31-M-12, symbol Connector:USB_C_Receptacle_USB2.0
- added R4, R5: 5.1k, Resistor_SMD:R_0805_2012Metric, symbol Device:R_Small
- added U1: ATmega32U2-AU, Package_QFP:TQFP-32_7x7mm_P0.8mm, symbol MCU_Microchip_ATmega:ATmega32U2-AU
- added Y1: 16MHz, Crystal:Resonator_SMD_muRata_CSTxExxV-3Pin_3.0x1.1mm, symbol Device:Resonator_Small
- C1, C2, C3, C4, C5: renamed from C?; footprint (none) -> Capacitor_SMD:C_0805_2012Metric
- R1, R2, R3, R6: renamed from R?; footprint (none) -> Resistor_SMD:R_0805_2012Metric
- SW1: renamed from SW?; footprint (none) -> random-keyboard-parts:SKQG-1155865
Connections:
- net labels added: GNDPWR
- wire segments 65 -> 70
- no-connect marks 0 -> 14
Other:
- moved on the sheet: C1, C2, C3, C4, C5, D1, D2, D3, D4, MX1, MX2, MX3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

Commit message: latest version
Parts:
- removed C2, C3: 0.1uF, Capacitor_SMD:C_0805_2012Metric, symbol Device:C_Small
Changed lines of the file:
@@
 	4550 3000 4550 3150
-$Comp
-L Device:C_Small C2
-U 1 1 6128EFC8
-P 3850 4350
-F 0 "C2" H 3942 4396 50  0000 L CNN
-F 1 "0.1uF" H 3942 4305 50  0000 L CNN
-F 2 "Capacitor_SMD:C_0805_2012Metric" H 3850 4350 50  0001 C CNN
-F 3 "~" H 3850 4350 50  0001 C CNN
-	1    3850 4350
-	1    0    0    -1
-$EndComp
-$Comp
-L Device:C_Small C3
-U 1 1 6128F36D
-P 4200 4350
-F 0 "C3" H 4292 4396 50  0000 L CNN
-F 1 "0.1uF" H 4292 4305 50  0000 L CNN
-F 2 "Capacitor_SMD:C_0805_2012Metric" H 4200 4350 50  0001 C CNN
-F 3 "~" H 4200 4350 50  0001 C CNN
-	1    4200 4350
-	1    0    0    -1
-$EndComp
 $Comp
 L Device:C_Small C4
@@
 	1    0    0    -1
 $EndComp
-Wire Wire Line
-	3850 4250 4200 4250
-Connection ~ 4200 4250
-Wire Wire Line
-	4200 4250 4400 4250
 Connection ~ 4600 4250
 Wire Wire Line
 	4600 4250 4950 4250
-Wire Wire Line
-	3850 4450 4200 4450
-Connection ~ 4200 4450
-Wire Wire Line
-	4200 4450 4400 4450
 Connection ~ 4600 4450
 Wire Wire Line
@@
 Wire Wire Line
 	4400 4100 4400 4250
-Connection ~ 4400 4250
 Wire Wire Line
 	4400 4250 4600 4250
 Wire Wire Line
 	4400 4450 4400 4600
-Connection ~ 4400 4450
 Wire Wire Line
 	4400 4450 4600 4450

Commit message: refine the routing
Parts:
- removed J1: USB_C_Receptacle_USB2.0, Connector_USB:USB_C_Receptacle_HRO_TYPE-C-31-M-12, symbol Connector:USB_C_Receptacle_USB2.0
- added C2: 0.1uF, Capacitor_SMD:C_0805_2012Metric, symbol Device:C_Small
- added D9: PRTR5V0U2X, Package_TO_SOT_SMD:SOT-143, symbol Power_Protection:PRTR5V0U2X
- added R7: 22, Resistor_SMD:R_0805_2012Metric, symbol Device:R_Small
- added R8: 5.1k, Resistor_SMD:R_0805_2012Metric, symbol Device:R_Small
- added USB1: HRO-TYPE-C-31-M-12, Type-C:HRO-TYPE-C-31-M-12-Assembly, symbol Type-C:HRO-TYPE-C-31-M-12
- R5: value 5.1k -> 22
Connections:
- net +5V: now also R1.1, C2.1
- net D+: now also R5.1
- net D-: now also R7.1
- net GND: now also C2.2, R8.1, USB1.1 (GND), USB1.12 (GND), USB1.13 (SHIELD); no longer R1.1, R5.1
- net VCC: now reaches F1.2
- net VCC: now also USB1.11 (VBUS), USB1.2 (VBUS)
- net at R4.2: now also USB1.4 (CC1)
- net at R5.2: now also D9.2 (I/O1), USB1.6 (DP1), USB1.8 (DP2)
- new net: R8.2, USB1.10 (CC2)
- new net: D9.3 (I/O2), R7.2, USB1.5 (DN2), USB1.7 (DN1)
Other:
- moved on the sheet: F1

Commit message: update firmware
Parts:
- removed C1: 1uF, Capacitor_SMD:C_0805_2012Metric, symbol Device:C_Small
- removed C2, C4: 0.1uF, Capacitor_SMD:C_0805_2012Metric, symbol Device:C_Small
- removed C5: 10uF, Capacitor_SMD:C_0805_2012Metric, symbol Device:C_Small
- removed D9: PRTR5V0U2X, Package_TO_SOT_SMD:SOT-143, symbol Power_Protection:PRTR5V0U2X
- removed F1: 500mA, Fuse:Fuse_1206_3216Metric, symbol Device:Polyfuse_Small
- removed R1, R6: 10k, Resistor_SMD:R_0805_2012Metric, symbol Device:R_Small
- removed R2, R3, R5, R7: 22, Resistor_SMD:R_0805_2012Metric, symbol Device:R_Small
- removed R4, R8: 5.1k, Resistor_SMD:R_0805_2012Metric, symbol Device:R_Small
- removed SW1: SW_Push, random-keyboard-parts:SKQG-1155865, symbol Switch:SW_Push
- removed U1: ATmega32U2-AU, Package_QFP:TQFP-32_7x7mm_P0.8mm, symbol MCU_Microchip_ATmega:ATmega32U2-AU
- removed USB1: HRO-TYPE-C-31-M-12, Type-C:HRO-TYPE-C-31-M-12-Assembly, symbol Type-C:HRO-TYPE-C-31-M-12
- removed Y1: 16MHz, Crystal:Resonator_SMD_muRata_CSTxExxV-3Pin_3.0x1.1mm, symbol Device:Resonator_Small
- added U1: Elite-C-keebio_without_bottom_row, Keebio-Parts:Elite-C-ZigZag, symbol SMP-v.2-rescue:Elite-C-keebio_without_bottom_row
Connections:
- net COL0: now also U1.13 (10/PB6)
- net COL1: now also U1.14 (16/PB2)
- net COL2: now also U1.15 (14/PB3)
- net COL3: now also U1.16 (15/PB1)
- net GND: now also U1.3 (GND), U1.4 (GND)
- net ROW0: now also U1.18 (A1/PF6)
- net ROW1: now also U1.19 (A2/PF5)
- no-connect marks 14 -> 0

Commit message: pcb and plate finalize for v.4
Parts:
- removed D2, D4: D_Small, Diode_SMD:D_SOD-123, symbol Device:D_Small
- removed MX4: MX-NoLED, MX_Only:MXOnly-1U-NoLED, symbol SMP-v.2-rescue:MX-NoLED-MX_Alps_Hybrid
- added D7, D8, D9: D_Small, 8hands:D_DO-35_SOD27_P5.08mm_Horizontal, symbol Device:D_Small
- added H5, H6, H7, H8: MountingHole_Pad, MountingHole:MountingHole_3.2mm_M3_Pad, symbol Mechanical:MountingHole_Pad
- added MX7, MX9: MX-NoLED, MX_Only:MXOnly-1U-NoLED, symbol SMP-v.2-rescue:MX-NoLED-MX_Alps_Hybrid
- D1: footprint Diode_SMD:D_SOD-123 -> 8hands:D_DO-35_SOD27_P5.08mm_Horizontal
- D2: renamed from D5; footprint Diode_SMD:D_SOD-123 -> 8hands:D_DO-35_SOD27_P5.08mm_Horizontal
- D3: renamed from D6; footprint Diode_SMD:D_SOD-123 -> 8hands:D_DO-35_SOD27_P5.08mm_Horizontal
- D4: renamed from D3; footprint Diode_SMD:D_SOD-123 -> 8hands:D_DO-35_SOD27_P5.08mm_Horizontal
- D5: renamed from D7; footprint Diode_SMD:D_SOD-123 -> 8hands:D_DO-35_SOD27_P5.08mm_Horizontal
- D6: renamed from D8; footprint Diode_SMD:D_SOD-123 -> 8hands:D_DO-35_SOD27_P5.08mm_Horizontal
- U1: footprint Keebio-Parts:Elite-C-ZigZag -> Keebio-Parts:Elite-C-ZigZag_no-fsilks
- renumbered MX5 to MX4, MX6 to MX5, MX7 to MX6
Connections:
- net COL0: now also U1.8 (5/PC6), MX7.1 (COL); no longer U1.13 (10/PB6)
- net COL1: now also MX8.1 (COL), U1.7 (4/PD4); no longer U1.14 (16/PB2)
- net COL2: now also U1.6 (3/PD0), MX9.1 (COL); no longer U1.15 (14/PB3)
- net ROW0: now also U1.9 (6/PD7), D7.1 (K), D8.1 (K), D9.1 (K); no longer D4.1 (K), D5.1 (K), D6.1 (K), U1.18 (A1/PF6)
- net ROW1: now also D4.1 (K), D5.1 (K), D6.1 (K), U1.10 (7/PE6); no longer D1.1 (K), D2.1 (K), D3.1 (K), U1.19 (A2/PF5)
- net at MX8.2 (ROW): now also D8.2 (A)
- net ROW2: now reaches U1.11 (8/PB4)
- net ROW2: now also D1.1 (K), D2.1 (K), D3.1 (K)
- net COL3: no longer names the net of U1.16 (15/PB1)
- net COL3: no longer MX8.1 (COL)
- new net: D7.2 (A), MX7.2 (ROW)
- new net: D9.2 (A), MX9.2 (ROW)
Other:
- moved on the sheet: H1, H2, H3, H4
