File: pcb/SMP v.2.sch (KiCad schematic (older format))
At the start: 27 parts, among them U1 Elite-C-keebio_without_bottom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

Commit message: add top plate
Parts:
- removed H5, H6, H7, H8: MountingHole_Pad, MountingHole:MountingHole_3.2mm_M3_Pad, symbol Mechanical:MountingHole_Pad
- MX1, MX2, MX3, MX4, MX5, MX6, MX7, MX8, MX9: footprint MX_Only:MXOnly-1U-NoLED -> MX_Only:MXOnly-1U-Hotswap
Changed lines of the file:
@@
 F 0 "MX1" H 8733 2723 60  0000 C CNN
 F 1 "MX-NoLED" H 8733 2649 20  0000 C CNN
-F 2 "MX_Only:MXOnly-1U-NoLED" H 8075 2475 60  0001 C CNN
+F 2 "MX_Only:MXOnly-1U-Hotswap" H 8075 2475 60  0001 C CNN
 F 3 "" H 8075 2475 60  0001 C CNN
 	1    8700 2500
@@
 F 0 "MX2" H 9333 2723 60  0000 C CNN
 F 1 "MX-NoLED" H 9333 2649 20  0000 C CNN
-F 2 "MX_Only:MXOnly-1U-NoLED" H 8675 2475 60  0001 C CNN
+F 2 "MX_Only:MXOnly-1U-Hotswap" H 8675 2475 60  0001 C CNN
 F 3 "" H 8675 2475 60  0001 C CNN
 	1    9300 2500
@@
 F 0 "MX3" H 9933 2723 60  0000 C CNN
 F 1 "MX-NoLED" H 9933 2649 20  0000 C CNN
-F 2 "MX_Only:MXOnly-1U-NoLED" H 9275 2475 60  0001 C CNN
+F 2 "MX_Only:MXOnly-1U-Hotswap" H 9275 2475 60  0001 C CNN
 F 3 "" H 9275 2475 60  0001 C CNN
 	1    9900 2500
@@
 F 0 "MX4" H 8733 3523 60  0000 C CNN
 F 1 "MX-NoLED" H 8733 3449 20  0000 C CNN
-F 2 "MX_Only:MXOnly-1U-NoLED" H 8075 3275 60  0001 C CNN
+F 2 "MX_Only:MXOnly-1U-Hotswap" H 8075 3275 60  0001 C CNN
 F 3 "" H 8075 3275 60  0001 C CNN
 	1    8700 3300
@@
 F 0 "MX5" H 9333 3523 60  0000 C CNN
 F 1 "MX-NoLED" H 9333 3449 20  0000 C CNN
-F 2 "MX_Only:MXOnly-1U-NoLED" H 8675 3275 60  0001 C CNN
+F 2 "MX_Only:MXOnly-1U-Hotswap" H 8675 3275 60  0001 C CNN
 F 3 "" H 8675 3275 60  0001 C CNN
 	1    9300 3300
@@
 F 0 "MX6" H 9933 3523 60  0000 C CNN
 F 1 "MX-NoLED" H 9933 3449 20  0000 C CNN
-F 2 "MX_Only:MXOnly-1U-NoLED" H 9275 3275 60  0001 C CNN
+F 2 "MX_Only:MXOnly-1U-Hotswap" H 9275 3275 60  0001 C CNN
 F 3 "" H 9275 3275 60  0001 C CNN
 	1    9900 3300
@@
 F 0 "MX7" H 8733 4323 60  0000 C CNN
 F 1 "MX-NoLED" H 8733 4249 20  0000 C CNN
-F 2 "MX_Only:MXOnly-1U-NoLED" H 8075 4075 60  0001 C CNN
+F 2 "MX_Only:MXOnly-1U-Hotswap" H 8075 4075 60  0001 C CNN
 F 3 "" H 8075 4075 60  0001 C CNN
 	1    8700 4100
@@
 F 0 "MX8" H 9333 4323 60  0000 C CNN
 F 1 "MX-NoLED" H 9333 4249 20  0000 C CNN
-F 2 "MX_Only:MXOnly-1U-NoLED" H 8675 4075 60  0001 C CNN
+F 2 "MX_Only:MXOnly-1U-Hotswap" H 8675 4075 60  0001 C CNN
 F 3 "" H 8675 4075 60  0001 C CNN
 	1    9300 4100
@@
 F 0 "MX9" H 9933 4323 60  0000 C CNN
 F 1 "MX-NoLED" H 9933 4249 20  0000 C CNN
-F 2 "MX_Only:MXOnly-1U-NoLED" H 9275 4075 60  0001 C CNN
+F 2 "MX_Only:MXOnly-1U-Hotswap" H 9275 4075 60  0001 C CNN
 F 3 "" H 9275 4075 60  0001 C CNN
 	1    9900 4100
@@
 Text GLabel 5300 2400 0    50   Input ~ 0
 COL2
-$Comp
-L Mechanical:MountingHole_Pad H5
-U 1 1 614B9DCF
-P 3800 3800
-F 0 "H5" H 3900 3849 50  0000 L CNN
-F 1 "MountingHole_Pad" H 3900 3758 50  0000 L CNN
-F 2 "MountingHole:MountingHole_3.2mm_M3_Pad" H 3800 3800 50  0001 C CNN
-F 3 "~" H 3800 3800 50  0001 C CNN
-	1    3800 3800
-	1    0    0    -1
-$EndComp
-$Comp
-L Mechanical:MountingHole_Pad H6
-U 1 1 614B9DD5
-P 3800 4100
-F 0 "H6" H 3900 4149 50  0000 L CNN
-F 1 "MountingHole_Pad" H 3900 4058 50  0000 L CNN
-F 2 "MountingHole:MountingHole_3.2mm_M3_Pad" H 3800 4100 50  0001 C CNN
-F 3 "~" H 3800 4100 50  0001 C CNN
-	1    3800 4100
-	1    0    0    -1
-$EndComp
-$Comp
-L Mechanical:MountingHole_Pad H7
-U 1 1 614B9DDB
-P 3800 4400
-F 0 "H7" H 3900 4449 50  0000 L CNN
-F 1 "MountingHole_Pad" H 3900 4358 50  0000 L CNN
-F 2 "MountingHole:MountingHole_3.2mm_M3_Pad" H 3800 4400 50  0001 C CNN
-F 3 "~" H 3800 4400 50  0001 C CNN
-	1    3800 4400
-	1    0    0    -1
-$EndComp
-$Comp
-L Mechanical:MountingHole_Pad H8
-U 1 1 614B9DE1
-P 3800 4700
-F 0 "H8" H 3900 4749 50  0000 L CNN
-F 1 "MountingHole_Pad" H 3900 4658 50  0000 L CNN
-F 2 "MountingHole:MountingHole_3.2mm_M3_Pad" H 3800 4700 50  0001 C CNN
-F 3 "~" H 3800 4700 50  0001 C CNN
-	1    3800 4700
-	1    0    0    -1
-$EndComp
 $EndSCHEMATC

Commit message: update pcb sch
Connections:
- net ROW0: now also D1.1 (K), D2.1 (K), D3.1 (K), U1.11 (8/PB4); no longer D7.1 (K), D8.1 (K), D9.1 (K), U1.9 (6/PD7)
- net ROW2: now also D7.1 (K), D8.1 (K), D9.1 (K), U1.9 (6/PD7); no longer D1.1 (K), D2.1 (K), D3.1 (K), U1.11 (8/PB4)
Changed lines of the file:
@@
 Wire Wire Line
 	10050 2450 10050 3250
-Text GLabel 8100 2850 0    50   Input ~ 0
+Text GLabel 8100 4450 0    50   Input ~ 0
 ROW2
 $Comp
@@
 Wire Wire Line
 	8850 3250 8850 4050
-Text GLabel 8100 4450 0    50   Input ~ 0
+Text GLabel 8100 2850 0    50   Input ~ 0
 ROW0
-Text GLabel 5300 2900 0    50   Input ~ 0
+Text GLabel 5300 2700 0    50   Input ~ 0
 ROW2
 Text GLabel 5300 2800 0    50   Input ~ 0
 ROW1
-Text GLabel 5300 2700 0    50   Input ~ 0
+Text GLabel 5300 2900 0    50   Input ~ 0
 ROW0
 Text GLabel 5300 2600 0    50   Input ~ 0
